File: KiCAD/LCDdisplayController.kicad_sch (KiCad schematic)
At the start: 19 parts, among them J1 Data_In0, J2 Data_In1, J3 LCD Connector, J4 LCD Connector, J5 Cond, U1 74HCT573, U2 74HCT573, U3 ATmega328-P, Y1 16MHz

Commit message: Updates of KiCad files and README
Parts:
- DS1: OrderInfo (none) -> https://www.amazon.com/gp/product/B0BFDGTPBP/ref=ox_sc_act_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; OrderInfo2 (none) -> https://www.amazon.com/dp/B0BFDDZ49T?ref=ppx_yo2ov_dt_b_fed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
- J1, J2: OrderInfo (none) -> https://www.digikey.com/en/products/detail/harwin-inc/M20-9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
- J3: OrderInfo (none) -> https://www.digikey.com/en/products/detail/w%C3%BCrth-elekt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
- J5: OrderInfo https://www.digikey.com/en/products/detail/sullins-connecto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 -> https://www.digikey.com/en/products/detail/metz-connect-usa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
- RV1: OrderInfo (none) -> https://www.digikey.com/en/products/detail/bourns-inc/PV37W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
- U2: OrderInfo (none) -> https://www.digikey.com/en/products/detail/texas-instrument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
Other:
- moved on the sheet: DS1
Changed lines of the file:
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@@
 			)
 		)
-		(property "OrderInfo" "https://www.digikey.com/en/products/detail/sullins-connector-solutions/PPTC061LFBN-RC/810145"
+		(property "OrderInfo" "https://www.digikey.com/en/products/detail/metz-connect-usa-inc/PR20206VBNN/12342874"
 			(at 204.47 90.17 0)
 			(effects
@@
 			)
 		)
+		(property "OrderInfo" "https://www.digikey.com/en/products/detail/w%C3%BCrth-elektronik/61301611821/6137797"
+			(at 209.55 50.8 0)
+			(effects
+				(font
+					(size 1.27 1.27)
+				)
+				(hide yes)
+			)
+		)
 		(pin "5"
 		)
@@
 			)
 		)
-		(property "OrderInfo" ""
+		(property "OrderInfo" "https://www.digikey.com/en/products/detail/harwin-inc/M20-9771146/3920928"
 			(at 27.94 87.63 0)
 			(effects
@@
 					(size 1.27 1.27)
 				)
+				(hide yes)
 			)
 		)
@@
 			)
 		)
+		(property "OrderInfo" "https://www.digikey.com/en/products/detail/bourns-inc/PV37W103C01B00/666597"
+			(at 161.29 38.1 0)
+			(effects
+				(font
+					(size 1.27 1.27)
+				)
+				(hide yes)
+			)
+		)
 		(pin "3"
 		)
@@
 			)
 		)
-		(property "OrderInfo" ""
+		(property "OrderInfo" "https://www.digikey.com/en/products/detail/harwin-inc/M20-9771146/3920928"
 			(at 27.94 161.29 0)
 			(effects
@@
 					(size 1.27 1.27)
 				)
+				(hide yes)
 			)
 		)
@@
 	(symbol
 		(lib_id "Display_Character:WC1602A")
-		(at 270.51 139.7 0)
+		(at 265.43 81.28 0)
 		(unit 1)
 		(exclude_from_sim no)
@@
 		(fields_autoplaced yes)
 		(property "Reference" "DS1"
-			(at 272.6533 116.84 0)
+			(at 267.5733 58.42 0)
 			(effects
 				(font
@@
 		)
 		(property "Value" "WC1602A"
-			(at 272.6533 119.38 0)
+			(at 267.5733 60.96 0)
 			(effects
 				(font
@@
 		)
 		(property "Footprint" "Display:WC1602A"
-			(at 270.51 162.56 0)
+			(at 265.43 104.14 0)
 			(effects
 				(font
@@
 		)
 		(property "Datasheet" "http://www.wincomlcd.com/pdf/WC1602A-SFYLYHTC06.pdf"
-			(at 288.29 139.7 0)
+			(at 283.21 81.28 0)
 			(effects
 				(font
@@
 		)
 		(property "Description" "LCD 16x2 Alphanumeric , 8 bit parallel bus, 5V VDD"
-			(at 270.51 139.7 0)
+			(at 265.43 81.28 0)
+			(effects
+				(font
+					(size 1.27 1.27)
+				)
+				(hide yes)
+			)
+		)
+		(property "OrderInfo" "https://www.amazon.com/gp/product/B0BFDGTPBP/ref=ox_sc_act_title_1?smid=A2RJ79XBQX6W3M&th=1"
+			(at 265.43 81.28 0)
+			(effects
+				(font
+					(size 1.27 1.27)
+				)
+				(hide yes)
+			)
+		)
+		(property "OrderInfo2" "https://www.amazon.com/dp/B0BFDDZ49T?ref=ppx_yo2ov_dt_b_fed_asin_title&th=1"
+			(at 265.43 81.28 0)
 			(effects
 				(font
@@
 			(at 58.42 163.83 0)
 			(effects
+				(font
+					(size 1.27 1.27)
+				)
+				(hide yes)
+			)
+		)
+		(property "OrderInfo" "https://www.digikey.com/en/products/detail/texas-instruments/CD74HCT573E/38717 "
+			(at 58.42 163.83 0)
+			(effects
