File: KiCAD/LCDdisplayController.kicad_pcb (KiCad board)
At the start: 2 copper layers, 99.1 x 77.5 mm, 18 parts, among them J1 Data_In0, J2 Data_In1, J3 LCD Connector, J4 LCD Connector, J5 Cond, U1 74HCT573, U2 74HCT573, U3 ATmega328-P, Y1 16MHz

Commit message: Updates of KiCad files and README
Parts:
- moved J1 1.27 mm to (43.2, 108.0)
- moved J5 1.27 mm to (80.0, 108.0)
Routing:
- net +5V: track 256.9 -> 257.9 mm
- net Net-(J1-Pin_4): track 5.08 -> 5.61 mm
- net Net-(J1-Pin_3): track 5.08 -> 5.61 mm
- net Net-(J1-Pin_2): track 5.08 -> 5.61 mm
- net /IN1: track 18.1 -> 17.6 mm
- net Net-(J1-Pin_9): track 5.08 -> 5.61 mm
- net Net-(J1-Pin_8): track 5.08 -> 5.61 mm
- net Net-(J1-Pin_7): track 5.08 -> 5.61 mm
- net Net-(J1-Pin_6): track 5.08 -> 5.61 mm
- net Net-(J1-Pin_5): track 5.08 -> 5.61 mm
- net /IN2: track 21.9 -> 21.4 mm
Other:
- outline, holes or cut-outs redrawn

Commit message: Some corrections
Routing:
- net GND: track 329.0 -> 331.5 mm
- net +5V: track 257.9 -> 259.4 mm
- net Net-(U1-Q0): track 109.0 -> 107.7 mm
- net Net-(U1-Q5): track 71.9 -> 70.7 mm
- net Net-(J2-Pin_10): track 31.8 -> 32.8 mm
Other:
- outline, holes or cut-outs redrawn
